Commit message: Adding righ hand pad -- Modifying the base_link.stl file of the right hand (Complete implementation)

File: talos_description/urdf/gripper/gripper.urdf.xacro (robot description, xacro)
@@ -11,5 +11,5 @@
                 <origin xyz="0 0 0" rpy="0 0 0" />
                 <geometry>
-                  <mesh filename="package://talos_description/meshes/gripper/base_link.STL" scale="1 1 1"/>
+                  <mesh filename="package://talos_description/meshes/gripper/base_link_pad.stl" scale="1 1 1"/>
                 </geometry>
                 <material name="DarkGrey"/>

File: talos_description/urdf/gripper/removeRightGripper.urdf.xacro (robot description, xacro)
@@ -11,5 +11,5 @@
                 <origin xyz="0 0 0" rpy="0 0 0" />
                 <geometry>
-                  <mesh filename="package://talos_description/meshes/gripper/base_link.STL" scale="1 1 1"/>
+                  <mesh filename="package://talos_description/meshes/gripper/base_link_pad.stl" scale="1 1 1"/>
                 </geometry>
                 <material name="DarkGrey"/>
@@ -18,5 +18,5 @@
                 <origin xyz="0 0 0" rpy="0 0 0" />
                 <geometry>
-                  <mesh filename="package://talos_description/meshes/gripper/base_link_collision.STL" scale="1 1 1"/>
+                  <mesh filename="package://talos_description/meshes/gripper/base_link_pad.stl" scale="1 1 1"/>
                 </geometry>
               </collision>
@@ -31,5 +31,5 @@
             <link name="${name}_motor_double_link">
               <xacro:call macro="${name}_motor_double_link_inertial" />
-              <visual>
+              <!-- <visual>
                 <origin xyz="-0.008 -0.02 -0.038" rpy="0 0 0" />
                 <geometry>
@@ -39,9 +39,9 @@
               </visual>
               <collision>
-                <origin xyz="0 0 0" rpy="0 0 0" />
+                <origin xyz="-0.008 -0.02 -0.038" rpy="0 0 0" />
                 <geometry>
                   <mesh filename="package://talos_description/meshes/gripper/pad.stl" scale="0.001 0.001 0.001"/>
                 </geometry>
-              </collision>
+              </collision> -->
               <!-- <visual>
                 <origin xyz="0 0 0" rpy="0 0 0" />
@@ -58,5 +58,5 @@
               </collision> -->
             </link>
-            <joint name="${name}_joint" type="revolute">
+            <!-- <joint name="${name}_joint" type="fixed">
               <parent link="${name}_base_link"/>
               <child link="${name}_motor_double_link"/>
@@ -64,4 +64,11 @@
                       rpy="${0.0 * deg_to_rad} ${0.0 * deg_to_rad} ${0.0 * deg_to_rad}"/>
               <axis xyz="1 0 0" />
+            </joint> -->
+            <joint name="${name}_joint" type="revolute">
+              <parent link="${name}_base_link"/>
+              <child link="${name}_motor_double_link"/>
+              <origin xyz="0.0 0.02025 -0.03"
+                      rpy="${0.0 * deg_to_rad} ${0.0 * deg_to_rad} ${0.0 * deg_to_rad}"/>
+              <axis xyz="1 0 0" />
               <limit lower="${-55.0 * deg_to_rad}" upper="${0.0 * deg_to_rad}" effort="1.0" velocity="1.0" />
               <dynamics friction="1.0" damping="1.0"/>
@@ -94,17 +101,4 @@
             <link name="${name}_fingertip_1_link">
               <xacro:call macro="${name}_fingertip_1_link_inertial" />
-              <visual>
-                <origin xyz="0 0 0" rpy="0 0 0" />
-                <geometry>
-                  <mesh filename="package://talos_description/meshes/gripper/slope_10deg.stl" scale="0.0001 0.0001 0.0001"/>
-                </geometry>
-              <material name="Orange"/>
-              </visual>
-              <collision>
-                <origin xyz="0 0 0" rpy="0 0 0" />
-                <geometry>
-                  <mesh filename="package://talos_description/meshes/gripper/slope_10deg.stl" scale="0.0001 0.0001 0.0001"/>
-                </geometry>
-              </collision>
               <!-- <visual>
                 <origin xyz="0 0 0" rpy="0 0 0" />

File: talos_description/urdf/talos_full_common.urdf.xacro (robot description, xacro)
@@ -20,4 +20,5 @@
   <xacro:include filename="$(find talos_description)/urdf/gripper/gripper.urdf.xacro" />
   <xacro:include filename="$(find talos_description)/urdf/gripper/removeRightGripper.urdf.xacro" />
+  <!-- <xacro:include filename="$(find talos_description)/urdf/gripper/pad.urdf.xacro" /> -->
   <xacro:include filename="$(find talos_description)/urdf/leg/leg.urdf.xacro" />
   <xacro:include filename="$(find talos_description)/urdf/leg/foot_collision_$(arg foot_collision).urdf.xacro" />
@@ -35,4 +36,5 @@
   <xacro:talos_gripper name="gripper_left" parent="wrist_left_ft_tool_link" reflect="1" />
   <xacro:talos_removeRightGripper name="gripper_right" parent="wrist_right_ft_tool_link" reflect="-1" />
+  <!-- <xacro:talos_pad name="pad_right" parent="gripper_right_base_link" reflect="-1" /> -->
   <xacro:talos_leg prefix="left"  reflect="1" flexibility="$(arg flexibility)"/>
   <xacro:talos_leg prefix="right" reflect="-1" flexibility="$(arg flexibility)"/>
